Commit message: Add 3-links hierarchy. Minor bug fixes

File: src/package_bot/urdf/robot.urdf (robot description, URDF)
Before this commit: robot RHexBot, 9 links, 8 joints
Links:
- added link hand_link_1, mass 1; collision box size=0.3 1 0.15; visual box size=0.3 1 0.15
- added link hand_link_2, mass 1; collision box size=0.3 1 0.15; visual box size=0.3 1 0.15
- added link hand_link_3, mass 1; collision box size=0.3 1 0.15; visual box size=0.3 1 0.15
Joints:
- added joint body_to_hand_1: type continuous, parent base_link, child hand_link_1, origin xyz=0 0 0.25 rpy=-2.8 0 0, axis 1 0 0
- added joint body_to_hand_2: type continuous, parent hand_link_1, child hand_link_2, origin xyz=0 -1 0 rpy=1.8 0 0, axis 1 0 0
- added joint body_to_hand_3: type continuous, parent hand_link_2, child hand_link_3, origin xyz=0 -1 0 rpy=-2 0 0, axis 1 0 0
